File: STM32G473VET_main_controller_board.kicad_pcb (KiCad board)
At the start: 4 copper layers, 60 x 40 mm, 174 parts, among them CN1 value, J1 SWD, J10 CAN2, J11 UART5, J12 UART1A, J16 Conn_01x03_MountingPin, J17 USB_B_Micro, J2 Conn_01x04_MountingPin, J7 RS-485, J8 CAN1, J9 CAN3, Q1 AO3400A, Q5 SSM3J332R, Q6 Q_PNP_BEC, Q7 Q_PNP_BEC, SW1 SW_Push_Dual_x2, SW2 SW_Push_Dual_x2, SW3 SW_Push_Dual_x2, SW4 SW_Push_Dual_x2, U1 W25N01GVZEIG, U10 RY3430, U11 RY8411, U12 TPD4E1U06DCKR, U13 RS3236, U14 TPD4E1U06DCKR, U15 TPD4E1U06DCKR, U16 CH343P, U18 TPD4E1U06DCKR, U2 STM32G473VETx, U3 LIS3MDLTR, U4 ICM-42688-P, U5 SN75176AD, U6 TCAN1042HVDR, U7 TCAN1042HVDR, U8 TCAN1042HVDR, U9 RS3236, Y1 3225 25MHz

Commit message: minor design adjustments
Routing:
- net Net-(U11-BS): track 0.00 -> 1.62 mm
Changed lines of the file:
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@@
 		(net "Net-(U16-VBUS)")
+	)
+	(segment
+		(start 86.829657 78.505684)
+		(end 87.171613 78.163728)
+		(width 0.5)
+		(layer "B.Cu")
+		(net "Net-(U11-BS)")
+	)
+	(segment
+		(start 85.691613 78.505684)
+		(end 86.829657 78.505684)
+		(width 0.5)
+		(layer "B.Cu")
+		(net "Net-(U11-BS)")
 	)
 	(via
@@
 	)
 	(zone
-		(net "Net-(D2-K)")
-		(layer "B.Cu")
-		(hatch edge 0.5)
-		(priority 23)
-		(connect_pads yes
-			(clearance 0.2)
-		)
-		(min_thickness 0.25)
-		(fill yes
-			(thermal_gap 0.5)
-			(thermal_bridge_width 0.5)
-			(island_removal_mode 1)
-		)
-		(polygon
-			(pts
-				(xy 86.439376 48.69) (xy 89.31 48.69) (xy 89.31 50.699091) (xy 86.44062 50.700868)
-			)
-		)
-	)
-	(zone
-		(net "+5V")
-		(layer "B.Cu")
-		(hatch edge 0.5)
-		(priority 25)
-		(connect_pads yes
-			(clearance 0.2)
-		)
-		(min_thickness 0.25)
-		(fill yes
-			(thermal_gap 0.5)
-			(thermal_bridge_width 0.5)
-			(island_removal_mode 0)
-		)
-		(polygon
-			(pts
-				(xy 128.3 54.3) (xy 129.2 54.3) (xy 130.6 55.8) (xy 130.6 56.8) (xy 129.6 56.8) (xy 129.6 56.0875)
-				(xy 128.9 55.3) (xy 128.3 55.3)
-			)
-		)
-	)
-	(zone
-		(net "VBATT+")
-		(layer "B.Cu")
-		(hatch edge 0.5)
-		(priority 7)
-		(connect_pads yes
-			(clearance 0.2)
-		)
-		(min_thickness 0.2)
-		(fill yes
-			(thermal_gap 0.5)
-			(thermal_bridge_width 0.5)
-			(island_removal_mode 0)
-		)
-		(polygon
-			(pts
-				(xy 79.5 72.55) (xy 86.75 72.55) (xy 86.75 68.25) (xy 75.75 68.25) (xy 75.75 74.175) (xy 79.5 74.175)
-			)
-		)
-	)
-	(zone
-		(net "+5V")
-		(layer "B.Cu")
-		(hatch edge 0.5)
-		(priority 17)
-		(connect_pads yes
-			(clearance 0.2)
-		)
-		(min_thickness 0.25)
-		(fill yes
-			(thermal_gap 0.5)
-			(thermal_bridge_width 0.5)
-			(island_removal_mode 1)
-		)
-		(polygon
-			(pts
-				(xy 107.7 49.1) (xy 109.5 49.1) (xy 109.5 48.4) (xy 110.7 48.4) (xy 110.7 49.8) (xy 111 49.8) (xy 111 52)
-				(xy 107.7 52) (xy 107.7 51) (xy 109.3 51) (xy 109.3 50.1) (xy 107.7 50.1)
-			)
-		)
-	)
-	(zone
 		(layer "B.Cu")
 		(hatch edge 0.5)
@@
 		(polygon
 			(pts
-				(xy 96.750565 79.010008) (xy 97.199996 79.010008) (xy 97.20005 80.099834) (xy 96.748815 80.099131)
-			)
-		)
-	)
-	(zone
-		(net "+3V3_IO")
-		(layer "B.Cu")
-		(hatch edge 0.5)
-		(priority 21)
-		(connect_pads yes
-			(clearance 0.2)
-		)
-		(min_thickness 0.25)
-		(fill yes
-			(thermal_gap 0.5)
-			(thermal_bridge_width 0.5)
-			(island_removal_mode 0)
-		)
-		(polygon
-			(pts
-				(xy 103.8 48.7) (xy 103.7 56.1) (xy 105.2 56.1) (xy 105.2 54.9) (xy 104.7 54.5) (xy 104.7 52.2)
-				(xy 105 52.2) (xy 105 49.9) (xy 106.9 49.9) (xy 106.9 49.3) (xy 105.1 49.3) (xy 105.1 48.7)
-			)
-		)
-	)
-	(zone
-		(net "Net-(U10-FB)")
-		(layer "B.Cu")
-		(hatch edge 0.5)
-		(priority 24)
+				(xy 99.9 72.124431) (xy 99.9 71.600028) (xy 100.989943 71.599974) (xy 100.989123 72.126181)
+			)
+		)
+	)
+	(zone
+		(net "Net-(D2-K)")
+		(layer "B.Cu")
+		(hatch edge 0.5)
+		(priority 23)
 		(connect_pads yes
 			(clearance 0.2)
@@
 		(polygon
 			(pts
-				(xy 94.57 79.07) (xy 93.14 79.07) (xy 93.14 77.61) (xy 92.999863 77.60998) (xy 93 76.66) (xy 94.35 76.66)
-				(xy 94.35 75.07) (xy 95.45 75.07) (xy 95.45 77.54) (xy 94.57 77.54)
+				(xy 86.439376 48.69) (xy 89.31 48.69) (xy 89.31 50.699091) (xy 86.44062 50.700868)
 			)
 		)
@@
 		(layer "B.Cu")
 		(hatch edge 0.5)
-		(priority 18)
+		(priority 25)
+		(connect_pads yes
+			(clearance 0.2)
+		)
+		(min_thickness 0.25)
+		(fill yes
+			(thermal_gap 0.5)
+			(thermal_bridge_width 0.5)
+			(island_removal_mode 0)
+		)
+		(polygon
+			(pts
+				(xy 128.3 54.3) (xy 129.2 54.3) (xy 130.6 55.8) (xy 130.6 56.8) (xy 129.6 56.8) (xy 129.6 56.0875)
+				(xy 128.9 55.3) (xy 128.3 55.3)
+			)
+		)
+	)
+	(zone
+		(net "VBATT+")
+		(layer "B.Cu")
+		(hatch edge 0.5)
+		(priority 7)
+		(connect_pads yes
+			(clearance 0.2)
+		)
+		(min_thickness 0.2)
+		(fill yes
+			(thermal_gap 0.5)
+			(thermal_bridge_width 0.5)
+			(island_removal_mode 0)
+		)
+		(polygon
+			(pts
+				(xy 79.5 72.55) (xy 86.75 72.55) (xy 86.75 68.25) (xy 75.75 68.25) (xy 75.75 74.175) (xy 79.5 74.175)
+			)
+		)
+	)
+	(zone
+		(net "+5V")
+		(layer "B.Cu")
+		(hatch edge 0.5)
+		(priority 17)
 		(connect_pads yes
 			(clearance 0.2)
@@
 		(polygon
 			(pts
-				(xy 93.13 48.6) (xy 93.13 50.6) (xy 90.5 50.6) (xy 90.5 52.5) (xy 92.8 52.5) (xy 92.8 53.3) (xy 89.7 53.3)
-				(xy 89.7 48.6)
-			)
-		)
-	)
-	(zone
-		(net "+5V")
-		(layer "B.Cu")
-		(hatch edge 0.5)
-		(priority 5)
-		(connect_pads yes
-			(clearance 0.2)
-		)
-		(min_thickness 0.2)
-		(fill yes
-			(thermal_gap 0.5)
-			(thermal_bridge_width 0.5)
-			(island_removal_mode 0)
-		)
-		(polygon
-			(pts
-				(xy 94.5 80.2) (xy 94.5 81.3) (xy 93.8 81.3) (xy 93.8 84.9) (xy 95 84.9) (xy 95 85.8) (xy 93.1 85.8)
-				(xy 93.1 86.6) (xy 91.5 86.6) (xy 91.5 85.8) (xy 91.5 84.4) (xy 92.7 84.4) (xy 92.7 80.2)
-			)
-		)
-	)
-	(zone
-		(net "Net-(U10-SW)")
-		(layer "B.Cu")
-		(hatch edge 0.5)
-		(priority 3)
-		(connect_pads yes
-			(clearance 0.15)
-		)
-		(min_thickness 0.2)
-		(fill yes
-			(thermal_gap 0.5)
-			(thermal_bridge_width 0.5)
-			(island_removal_mode 0)
-		)
-		(polygon
-			(pts
-				(xy 95.637499 80.31) (xy 97.087499 80.31) (xy 98.981566 82.204067) (xy 98.981566 83.284067) (xy 98.401566 83.284067)
-				(xy 95.637499 80.52)
+				(xy 107.7 49.1) (xy 109.5 49.1) (xy 109.5 48.4) (xy 110.7 48.4) (xy 110.7 49.8) (xy 111 49.8) (xy 111 52)
+				(xy 107.7 52) (xy 107.7 51) (xy 109.3 51) (xy 109.3 50.1) (xy 107.7 50.1)
 			)
 		)
@@
 		(placement
 			(enabled no)
+			(sheetname "/")
+		)
+		(fill
+			(thermal_gap 0.5)
+			(thermal_bridge_width 0.5)
+			(island_removal_mode 0)
+		)
+		(polygon
+			(pts
+				(xy 96.750565 79.010008) (xy 97.199996 79.010008) (xy 97.20005 80.099834) (xy 96.748815 80.099131)
+			)
+		)
+	)
+	(zone
+		(net "+3V3_IO")
+		(layer "B.Cu")
+		(hatch edge 0.5)
+		(priority 21)
+		(connect_pads yes
+			(clearance 0.2)
+		)
+		(min_thickness 0.25)
+		(fill yes
+			(thermal_gap 0.5)
+			(thermal_bridge_width 0.5)
+			(island_removal_mode 0)
+		)
+		(polygon
+			(pts
+				(xy 103.8 48.7) (xy 103.7 56.1) (xy 105.2 56.1) (xy 105.2 54.9) (xy 104.7 54.5) (xy 104.7 52.2)
+				(xy 105 52.2) (xy 105 49.9) (xy 106.9 49.9) (xy 106.9 49.3) (xy 105.1 49.3) (xy 105.1 48.7)
+			)
+		)
+	)
+	(zone
+		(net "Net-(U10-FB)")
+		(layer "B.Cu")
+		(hatch edge 0.5)
+		(priority 24)
+		(connect_pads yes
+			(clearance 0.2)
+		)
+		(min_thickness 0.25)
+		(fill yes
+			(thermal_gap 0.5)
+			(thermal_bridge_width 0.5)
+			(island_removal_mode 1)
+		)
+		(polygon
+			(pts
+				(xy 94.57 79.07) (xy 93.14 79.07) (xy 93.14 77.61) (xy 92.999863 77.60998) (xy 93 76.66) (xy 94.35 76.66)
+				(xy 94.35 75.07) (xy 95.45 75.07) (xy 95.45 77.54) (xy 94.57 77.54)
+			)
+		)
+	)
+	(zone
+		(net "+5V")
+		(layer "B.Cu")
+		(hatch edge 0.5)
+		(priority 18)
+		(connect_pads yes
+			(clearance 0.2)
+		)
+		(min_thickness 0.25)
+		(fill yes
+			(thermal_gap 0.5)
+			(thermal_bridge_width 0.5)
+			(island_removal_mode 1)
+		)
+		(polygon
+			(pts
+				(xy 93.13 48.6) (xy 93.13 50.6) (xy 90.5 50.6) (xy 90.5 52.5) (xy 92.8 52.5) (xy 92.8 53.3) (xy 89.7 53.3)
+				(xy 89.7 48.6)
+			)
+		)
+	)
+	(zone
+		(net "+5V")
+		(layer "B.Cu")
+		(hatch edge 0.5)
+		(priority 5)
+		(connect_pads yes
+			(clearance 0.2)
+		)
+		(min_thickness 0.2)
+		(fill yes
+			(thermal_gap 0.5)
+			(thermal_bridge_width 0.5)
+			(island_removal_mode 0)
+		)
+		(polygon
+			(pts
+				(xy 94.5 80.2) (xy 94.5 81.3) (xy 93.8 81.3) (xy 93.8 84.9) (xy 95 84.9) (xy 95 85.8) (xy 93.1 85.8)
+				(xy 93.1 86.6) (xy 91.5 86.6) (xy 91.5 85.8) (xy 91.5 84.4) (xy 92.7 84.4) (xy 92.7 80.2)
+			)
+		)
+	)
+	(zone
+		(net "Net-(U10-SW)")
+		(layer "B.Cu")
+		(hatch edge 0.5)
+		(priority 3)
+		(connect_pads yes
+			(clearance 0.15)
+		)
+		(min_thickness 0.2)
+		(fill yes
+			(thermal_gap 0.5)
+			(thermal_bridge_width 0.5)
+			(island_removal_mode 0)
+		)
+		(polygon
+			(pts
+				(xy 95.637499 80.31) (xy 97.087499 80.31) (xy 98.981566 82.204067) (xy 98.981566 83.284067) (xy 98.401566 83.284067)
+				(xy 95.637499 80.52)
+			)
+		)
+	)
+	(zone
+		(layer "B.Cu")
+		(hatch edge 0.5)
+		(connect_pads yes
+			(clearance 0)
+		)
+		(min_thickness 0.25)
+		(keepout
+			(tracks allowed)
+			(vias allowed)
+			(pads allowed)
+			(copperpour not_allowed)
+			(footprints allowed)
+		)
+		(placement
+			(enabled no)
 			(sheetname "")
 		)
@@
 	)
 	(zone
+		(layer "B.Cu")
+		(hatch edge 0.5)
+		(connect_pads yes
+			(clearance 0)
+		)
+		(min_thickness 0.25)
+		(keepout
+			(tracks allowed)
+			(vias allowed)
+			(pads allowed)
+			(copperpour not_allowed)
+			(footprints allowed)
+		)
+		(placement
+			(enabled no)
+			(sheetname "/")
+		)
+		(fill
+			(thermal_gap 0.5)
+			(thermal_bridge_width 0.5)
+			(island_removal_mode 0)
+		)
+		(polygon
+			(pts
+				(xy 105.400884 73.8) (xy 105.7 73.8) (xy 105.700021 74.225233) (xy 105.400202 74.224765)
+			)
+		)
+	)
+	(zone
 		(net "+5V")
 		(layer "In1.Cu")
@@
 			(pts
 				(xy 117.75 52.5) (xy 117.75 54.75) (xy 116.1 56.4) (xy 108.29 56.4) (xy 99.12 65.57) (xy 99.12 79)
-				(xy 122.825 79) (xy 122.825 80) (xy 127.6 80) (xy 127.6 86.7) (xy 101.7 86.7) (xy 99.5 84.5) (xy 78.3 84.5)
+				(xy 122.825 79) (xy 122.825 80) (xy 127.4 80) (xy 127.4 86.7) (xy 101.7 86.7) (xy 99.5 84.5) (xy 78.3 84.5)
 				(xy 78.3 52.5)
 			)
